Commit message: Created core URDF

File: description/robot_core.xacro (robot description, xacro)
@@ -40,7 +40,4 @@
             <origin xyz="0.15 0 0.075" rpy="0 0 0"/>
         </xacro:inertial_box>
-        <gazebo reference="chassis">
-            <material>Gazebo/Red</material>
-        </gazebo>
     </link>
     <joint name="left_wheel_joint" type="continuous">
@@ -65,7 +62,4 @@
             <origin xyz="0 0 0" rpy="0 0 0"/>
         </xacro:inertial_cylinder>
-        <gazebo reference="right_wheel">
-            <material>Gazebo/Blue</material>
-        </gazebo>
     </link>
     <joint name="right_wheel_joint" type="continuous">
@@ -90,7 +84,4 @@
             <origin xyz="0 0 0" rpy="0 0 0"/>
         </xacro:inertial_cylinder>
-        <gazebo reference="right_wheel">
-            <material>Gazebo/Blue</material>
-        </gazebo>
     </link>
     <joint name="caster_wheel_joint" type="fixed">
@@ -115,8 +106,3 @@
         </xacro:inertial_sphere>
     </link>
-    <gazebo reference="caster_wheel">
-        <material>Gazebo/Black</material>
-        <mu1 value="0.001"/>
-        <mu2 value="0.001"/>
-    </gazebo>
 </robot>
